Commit message: Update youbot.urdf.xacro

File: youbot_description/robots/youbot.urdf.xacro (robot description, xacro)
@@ -39,5 +39,5 @@
   </xacro:youbot_arm>
   <xacro:new_gripper_urdf name="gripper" parent="arm_link_5">
-       <origin xyz="-0.00031 -0.01549 -0.017" rpy="0 0 -1.5708" />   <!--<origin xyz="-0.00031 -0.01549 -0.0225" rpy="0 0 -1.5708" /> -->
+       <origin xyz="-0.00031 -0.01549 -0.017" rpy="0 0 -1.5708" />
   </xacro:new_gripper_urdf>
   <!-- base laser front -->
